Commit message: Initialized Gazebo Simulation Setup

File: sAMR_description/urdf/materials.urdf.xacro (robot description, xacro)
@@ -1,3 +1,3 @@
-<robot xmlns:xacro="http://www.ros.org/wiki/xacro" name="axebot">
+<robot xmlns:xacro="http://www.ros.org/wiki/xacro" name="samr">
   <!-- Green material -->
   <material name="green">

File: sAMR_description/urdf/samr_core.xacro (robot description, xacro)
@@ -1,4 +1,4 @@
 <?xml version="1.0"?>
-<robot xmlns:xacro="http://www.ros.org/wiki/xacro" name="sAMR">
+<robot xmlns:xacro="http://www.ros.org/wiki/xacro" name="samr">
     <xacro:property name="PI" value="3.1415926535897931"/>
     <xacro:property name="chassis_radius" value="0.085"/>
@@ -7,4 +7,5 @@
     <xacro:include filename="$(find sAMR_description)/urdf/materials.urdf.xacro"/>
     <xacro:include filename="$(find sAMR_description)/urdf/wheel.urdf.xacro"/>
+    <xacro:include filename="$(find sAMR_description)/urdf/ros2_control.xacro"/>
     <link name="base_footprint"/>
     <joint name="base_joint" type="fixed">
@@ -17,28 +18,30 @@
             <origin xyz="0 0 0.0" rpy="0 0 ${PI/6}"/>
             <geometry>
-                <mesh filename="package://sAMR_description/meshes/baselink.stl" scale="0.001 0.001 0.001"/>
+                <mesh filename="file://$(find sAMR_description)/meshes/baselink.stl" scale="0.001 0.001 0.001"/>
             </geometry>
             <material name="white"/>
         </visual>
         <collision>
-            <origin xyz="0 0 0" rpy="0 0 0"/>
+            <origin xyz="0 0 0" rpy="0 0 ${PI/6}"/>
             <geometry>
-                <mesh filename="package://sAMR_description/meshes/baselink.stl" scale="0.001 0.001 0.001"/>
+                <mesh filename="file://$(find sAMR_description)/meshes/baselink.stl" scale="0.001 0.001 0.001"/>
             </geometry>
         </collision>
+        <inertial>
+            <origin xyz="-0.0058 -0.0034 -0.08134" rpy="0.0 0.0 0.0"/>
+            <mass value="2.428"/>
+            <inertia ixx="0.04625" ixy="0.000085" ixz="0.000287" iyy="0.04634" iyz="0.000166" izz="0.02341"/>
+        </inertial>
     </link>
-    <joint name="ball_joint" type="fixed">
+    <joint name="dummy_joint" type="fixed">
         <parent link="base_link"/>
-        <child link="ball_link"/>
-        <origin xyz="0.0 0.0 -0.2598" rpy="0.0 0.0 0.0"/>
+        <child link="dummy_link"/>
+        <origin xyz="-0.0058 -0.0034 -0.05365" rpy="0 0 0"/>
     </joint>
-    <link name="ball_link">
-        <visual>
-            <origin xyz="0.0 0.0 0.0" rpy="0.0 0.0 0.0"/>
+    <link name="dummy_link">
+        <origin xyz="-0.0058 -0.0034 -0.05365" rpy="0.0 0.0 0.0"/>
             <geometry>
-                <sphere radius="0.121"/>
+                <sphere radius="0.001"/>
             </geometry>
-            <material name="orange"/>
-        </visual>
     </link>
     <!-- Define wheels dynamically -->

File: sAMR_description/urdf/wheel.urdf.xacro (robot description, xacro)
@@ -15,12 +15,12 @@
                 <origin xyz="0.0 0.0 0.0" rpy="0.0 0.0 0.0"/>
                 <geometry>
-                    <mesh filename="package://sAMR_description/meshes/roller.stl" scale= "0.001 0.001 0.001"/>
+                    <mesh filename="file://$(find sAMR_description)/meshes/roller.stl" scale= "0.001 0.001 0.001"/>
                 </geometry>
-                <material name="black"/>
+                <material name="${material}"/>
             </visual>
             <collision>
                 <origin xyz="0.0 0.0 0.0" rpy="0.0 0.0 0.0"/>
                 <geometry>
-                    <mesh filename="package://sAMR_description/meshes/roller.stl" scale= "0.001 0.001 0.001"/>
+                    <mesh filename="file://$(find sAMR_description)/meshes/roller.stl" scale= "0.001 0.001 0.001"/>
                 </geometry>
             </collision>
@@ -59,5 +59,5 @@
                 <origin xyz="0.0 0.0 0.0" rpy="0.0 0.0 0.0"/>
                 <geometry>
-                    <mesh filename="package://sAMR_description/meshes/wheel.stl" scale="0.001 0.001 0.001"/>
+                    <mesh filename="file://$(find sAMR_description)/meshes/wheel.stl" scale="0.001 0.001 0.001"/>
                 </geometry>
                 <material name="${material}"/>
@@ -66,5 +66,5 @@
                 <origin xyz="0.0 0.0 0.0" rpy="0.0 0.0 0.0"/>
                 <geometry>
-                    <mesh filename="package://sAMR_description/meshes/wheel.stl" scale="0.001 0.001 0.001"/>
+                    <mesh filename="file://$(find sAMR_description)/meshes/wheel.stl" scale="0.001 0.001 0.001"/>
                 </geometry>
             </collision>
