Commit message: Renamed model description package name

File: description/urdf/samr_core.xacro (robot description, xacro)
@@ -5,7 +5,7 @@
     <xacro:property name="wheel_thickness" value="0.01905" />
     <xacro:property name="motor_shaft_length" value="0.005475"/>
-    <xacro:include filename="$(find sAMR_description)/urdf/materials.urdf.xacro"/>
-    <xacro:include filename="$(find sAMR_description)/urdf/wheel.urdf.xacro"/>
-    <xacro:include filename="$(find sAMR_description)/urdf/ros2_control.xacro"/>
+    <xacro:include filename="materials.urdf.xacro"/>
+    <xacro:include filename="wheel.urdf.xacro"/>
+    <xacro:include filename="ros2_control.xacro"/>
     <link name="base_footprint"/>
     <joint name="base_joint" type="fixed">
@@ -25,5 +25,5 @@
             <origin xyz="0 0 0" rpy="0 0 ${PI/6}"/>
             <geometry>
-                <mesh filename="file://$(find sAMR_description)/meshes/baselink.stl" scale="0.001 0.001 0.001"/>
+                <mesh filename="file://$(find sAMR_description)//meshes/baselink.stl" scale="0.001 0.001 0.001"/>
             </geometry>
         </collision>
@@ -34,5 +34,6 @@
         </inertial>
     </link>
-    <joint name="dummy_joint" type="fixed">
+    </robot>
+    <!-- <joint name="dummy_joint" type="fixed">
         <parent link="base_link"/>
         <child link="dummy_link"/>
@@ -45,5 +46,5 @@
             </geometry>
     </link>
-    <!-- Define wheels dynamically -->
+    Define wheels dynamically
     <xacro:wheel_macro suffix="1" theta="${PI}" chassis_radius="${chassis_radius}"
                     material="blue"/>
@@ -51,4 +52,3 @@
                     material="blue"/>
     <xacro:wheel_macro suffix="3" theta="${PI/3}" chassis_radius="${chassis_radius}"
-                    material="blue"/>
-</robot>
+                    material="blue"/> -->
